File: Kicad/navball_module.kicad_sch (KiCad schematic)
At the start: 4 parts, among them J2 Conn_01x13

Commit message: schematics correction
Parts:
- added C69: 22uF, Capacitor_SMD:C_1206_3216Metric_Pad1.33x1.80mm_HandSolder, symbol Device:C
- C31, C32, C33: LCSC Part (none) -> C14663; Manufacturer_Name (none) -> Yageo; Manufacturer_Part_Number (none) -> CC0603KRX7R9BB104
- J2: footprint Connector_JST:JST_GH_SM12B-GHS-TB_1x12-1MP_P1.25mm_Horizontal -> Connector_JST:JST_GH_SM13B-GHS-TB_1x13-1MP_P1.25mm_Horizontal; LCSC Part (none) -> C515957; Manufacturer_Name (none) -> JST; Manufacturer_Part_Number (none) -> SM13B-GHS-TB(LF)(SN)
Connections:
- net 3.3V: now also C69.1
- net GND: now also C69.2
Other:
- moved on the sheet: C31, C32, C33, J2
