File: Kicad/seg_4x14_module.kicad_sch (KiCad schematic)
At the start: 7 parts, among them U2 HT16K33A-28SSOP

Commit message: schematics correction
Parts:
- added C46, C52: 100n, Capacitor_SMD:C_0603_1608Metric_Pad1.08x0.95mm_HandSolder, symbol Device:C
- added C74: 22uF, Capacitor_SMD:C_1206_3216Metric_Pad1.33x1.80mm_HandSolder, symbol Device:C
- D1: value CUS530 -> SD103AWS; footprint (none) -> Diode_SMD:D_SOD-323_HandSoldering; LCSC Part (none) -> C181207; Manufacturer_Name (none) -> Guangdong Hottech; Manufacturer_Part_Number (none) -> SD103AWS
- LED26: renamed from LED1; footprint 4segment_x2:LED-SEG-TH_18P-L25.2-W21.1-P2.54-LS15.2-BL -> Eeloo_Pad:LED-SEG-TH_18P-L25.2-W21.1-P2.54-LS15.2-BL; Manufacturer_Name (none) -> ZHIHAO; Manufacturer_Part_Number (none) -> FJ5241AH
- LED27: renamed from LED7; footprint 4segment_x2:LED-SEG-TH_18P-L25.2-W21.1-P2.54-LS15.2-BL -> Eeloo_Pad:LED-SEG-TH_18P-L25.2-W21.1-P2.54-LS15.2-BL; Manufacturer_Name (none) -> ZHIHAO; Manufacturer_Part_Number (none) -> FJ5241AH
- R13: renamed from R11; footprint (none) -> Resistor_SMD:R_0603_1608Metric_Pad0.98x0.95mm_HandSolder; LCSC Part (none) -> C23153; Manufacturer_Name (none) -> UNI-ROYAL; Manufacturer_Part_Number (none) -> 0603WAF3902T5E
- R14: renamed from R17; footprint (none) -> Resistor_SMD:R_0603_1608Metric_Pad0.98x0.95mm_HandSolder; LCSC Part (none) -> C23153; Manufacturer_Name (none) -> UNI-ROYAL; Manufacturer_Part_Number (none) -> 0603WAF3902T5E
- R15: renamed from R23; footprint (none) -> Resistor_SMD:R_0603_1608Metric_Pad0.98x0.95mm_HandSolder; LCSC Part (none) -> C23153; Manufacturer_Name (none) -> UNI-ROYAL; Manufacturer_Part_Number (none) -> 0603WAF3902T5E
- U1: renamed from U2; footprint HT16K33A-28SSOP:SOP63P600X175-28N -> Eeloo_Pad:SOP63P600X175-28N; LCSC Part (none) -> C5444738; Manufacturer_Name (none) -> Holtek; Manufacturer_Part_Number (none) -> HT16K33A-28SSOP
Connections:
- net +5V: now also C46.1, C52.1, C74.1
- net GND: now also C46.2, C52.2, C74.2
