File: Kicad/uC1.kicad_sch (KiCad schematic)
At the start: 25 parts, among them IC1 W25Q16JVUXIQ_TR, J3 SC0914_13_, SW1 SW_Push, SW2 SW_Push, Y1 ABM8-272-T3

Commit message: schematics correction
Parts:
- C1, C10, C11, C12, C13, C14, C3, C4, C8, C9: LCSC Part (none) -> C14663; Manufacturer_Name (none) -> Yageo; Manufacturer_Part_Number (none) -> CC0603KRX7R9BB104
- C15: footprint Capacitor_SMD:C_0603_1608Metric_Pad1.08x0.95mm_HandSolder -> Capacitor_SMD:C_1206_3216Metric_Pad1.33x1.80mm_HandSolder; LCSC Part (none) -> C13585; Manufacturer_Name (none) -> Samsung Electro-Mechanics; Manufacturer_Part_Number (none) -> CL31A106KBHNNNE
- C2, C7: LCSC Part (none) -> C15849; Manufacturer_Name (none) -> Samsung Electro-Mechanics; Manufacturer_Part_Number (none) -> CL10A105KB8NNNC
- C5, C6: LCSC Part (none) -> C1644; Manufacturer_Name (none) -> Samsung Electro-Mechanics; Manufacturer_Part_Number (none) -> CL10C150JB8NNNC
- IC1: LCSC Part (none) -> C2843335
- J12: renamed from J3; LCSC Part (none) -> C2040; Manufacturer_Name RASPBERRY-PI -> Raspberry Pi
- R3: renamed from R1; LCSC Part (none) -> C21190; Manufacturer_Name (none) -> UNI-ROYAL; Manufacturer_Part_Number (none) -> 0603WAF1001T5E
- R5: renamed from R3; LCSC Part (none) -> C21190; Manufacturer_Name (none) -> UNI-ROYAL; Manufacturer_Part_Number (none) -> 0603WAF1001T5E
- R6: renamed from R4; value 27.2 -> 27.4; footprint Resistor_SMD:R_0603_1608Metric_Pad0.98x0.95mm_HandSolder -> Resistor_SMD:R_0402_1005Metric_Pad0.72x0.64mm_HandSolder; LCSC Part (none) -> C274349; Manufacturer_Name (none) -> Yageo; Manufacturer_Part_Number (none) -> RC0402FR-0727R4L
- R7: renamed from R5; value 27.2 -> 27.4; footprint Resistor_SMD:R_0603_1608Metric_Pad0.98x0.95mm_HandSolder -> Resistor_SMD:R_0402_1005Metric_Pad0.72x0.64mm_HandSolder; LCSC Part (none) -> C274349; Manufacturer_Name (none) -> Yageo; Manufacturer_Part_Number (none) -> RC0402FR-0727R4L
- SW1, SW2: footprint Button_Switch_SMD:SW_SPST_TL3305A -> Button_Switch_SMD:SW_Push_1P1T_XKB_TS-1187A; LCSC Part (none) -> C318884; Manufacturer_Name (none) -> XKB Connection; Manufacturer_Part_Number (none) -> TS-1187A-B-A-B
- Y1: LCSC Part (none) -> C20625731
- renumbered R2 to R4
