File: Kicad/Eeloo_Pad.kicad_pcb (KiCad board)
At the start: 2 copper layers, 100 parts, among them IC1 W25Q16JVUXIQ_TR, IC2 W25Q16JVUXIQ_TR, IC3 ADS1015IDGST, IC4 PCF8575DBQR, IC5 PCF8575DBQR, J1 USB_C_Receptacle_USB2.0_16P, J2 Conn_01x13, J3 SC0914_13_, J4 SC0914_13_, SW1 SW_Push, SW2 SW_Push, SW3 SW_Push, SW4 SW_Push, U1 HT16K33A-28SSOP, U2 HT16K33A-28SSOP, U3 HT16K33A-28SSOP, U4 HT16K33A-28SSOP, U5 HT16K33A-28SSOP, U6 HT16K33A-28SSOP, Y1 ABM8-272-T3, Y2 ABM8-272-T3

Commit message: schematics correction
Parts:
- added C34: 100n, Capacitor_SMD:C_0603_1608Metric_Pad1.08x0.95mm_HandSolder, F.Cu at (233.8, 15.9)
- added C35: 100n, Capacitor_SMD:C_0603_1608Metric_Pad1.08x0.95mm_HandSolder, F.Cu at (322.6, 61.8)
- added C36: 100n, Capacitor_SMD:C_0603_1608Metric_Pad1.08x0.95mm_HandSolder, F.Cu at (325.1, 61.8)
- added C37: 100n, Capacitor_SMD:C_0603_1608Metric_Pad1.08x0.95mm_HandSolder, F.Cu at (327.6, 61.8)
- added C38: 100n, Capacitor_SMD:C_0603_1608Metric_Pad1.08x0.95mm_HandSolder, F.Cu at (330.1, 61.8)
- added C39: 100n, Capacitor_SMD:C_0603_1608Metric_Pad1.08x0.95mm_HandSolder, F.Cu at (262.6, 58.1)
- added C40: 100n, Capacitor_SMD:C_0603_1608Metric_Pad1.08x0.95mm_HandSolder, F.Cu at (169.7, -4.14)
- added C41: 100n, Capacitor_SMD:C_0603_1608Metric_Pad1.08x0.95mm_HandSolder, F.Cu at (169.7, -1.63)
- added C42: 100n, Capacitor_SMD:C_0603_1608Metric_Pad1.08x0.95mm_HandSolder, F.Cu at (261.1, 58.1)
- added C43: 100n, Capacitor_SMD:C_0603_1608Metric_Pad1.08x0.95mm_HandSolder, F.Cu at (336.4, 41.8)
- added C44: 100n, Capacitor_SMD:C_0603_1608Metric_Pad1.08x0.95mm_HandSolder, F.Cu at (338.9, 41.8)
- added C45: 100n, Capacitor_SMD:C_0603_1608Metric_Pad1.08x0.95mm_HandSolder, F.Cu at (341.4, 41.8)
- added C46: 100n, Capacitor_SMD:C_0603_1608Metric_Pad1.08x0.95mm_HandSolder, F.Cu at (78.9, 79.8)
- added C47: 100n, Capacitor_SMD:C_0603_1608Metric_Pad1.08x0.95mm_HandSolder, F.Cu at (161.5, 85.6)
- added C48: 100n, Capacitor_SMD:C_0603_1608Metric_Pad1.08x0.95mm_HandSolder, F.Cu at (272.0, 86.6)
- added C49: 100n, Capacitor_SMD:C_0603_1608Metric_Pad1.08x0.95mm_HandSolder, F.Cu at (107.6, 86.5)
- added C50: 100n, Capacitor_SMD:C_0603_1608Metric_Pad1.08x0.95mm_HandSolder, F.Cu at (217.6, 86.7)
- added C51: 100n, Capacitor_SMD:C_0603_1608Metric_Pad1.08x0.95mm_HandSolder, F.Cu at (323.2, 86.4)
- added C52: 100n, Capacitor_SMD:C_0603_1608Metric_Pad1.08x0.95mm_HandSolder, F.Cu at (81.4, 79.8)
- added C53: 100n, Capacitor_SMD:C_0603_1608Metric_Pad1.08x0.95mm_HandSolder, F.Cu at (164.0, 85.6)
- added C54: 100n, Capacitor_SMD:C_0603_1608Metric_Pad1.08x0.95mm_HandSolder, F.Cu at (274.6, 86.6)
- added C55: 100n, Capacitor_SMD:C_0603_1608Metric_Pad1.08x0.95mm_HandSolder, F.Cu at (110.1, 86.5)
- added C56: 100n, Capacitor_SMD:C_0603_1608Metric_Pad1.08x0.95mm_HandSolder, F.Cu at (220.1, 86.7)
- added C57: 100n, Capacitor_SMD:C_0603_1608Metric_Pad1.08x0.95mm_HandSolder, F.Cu at (325.7, 86.4)
- added C58: 22uF, Capacitor_SMD:C_1206_3216Metric_Pad1.33x1.80mm_HandSolder, F.Cu at (76.3, 127.4)
- added C59: 22uF, Capacitor_SMD:C_1206_3216Metric_Pad1.33x1.80mm_HandSolder, F.Cu at (76.3, 122.3)
- added C60: 22uF, Capacitor_SMD:C_1206_3216Metric_Pad1.33x1.80mm_HandSolder, F.Cu at (78.6, 122.3)
- added C61: 100nF, Capacitor_SMD:C_0603_1608Metric_Pad1.08x0.95mm_HandSolder, F.Cu at (80.6, 128.3)
- added C62: 100nF, Capacitor_SMD:C_0603_1608Metric_Pad1.08x0.95mm_HandSolder, F.Cu at (84.8, 124.9)
- added C63: 100nF, Capacitor_SMD:C_0603_1608Metric_Pad1.08x0.95mm_HandSolder, F.Cu at (80.6, 121.5)
- added C64: 100n, Capacitor_SMD:C_0603_1608Metric_Pad1.08x0.95mm_HandSolder, F.Cu at (56.6, 134.2)
- added C65: 22uF, Capacitor_SMD:C_1206_3216Metric_Pad1.33x1.80mm_HandSolder, F.Cu at (78.6, 127.4)
- added C66: 22uF, Capacitor_SMD:C_1206_3216Metric_Pad1.33x1.80mm_HandSolder, F.Cu at (48.1, 121.0)
- added C67: 22uF, Capacitor_SMD:C_1206_3216Metric_Pad1.33x1.80mm_HandSolder, F.Cu at (47.8, 134.7)
- added C68: 22uF, Capacitor_SMD:C_1206_3216Metric_Pad1.33x1.80mm_HandSolder, F.Cu at (52.0, 123.8)
- added C69: 22uF, Capacitor_SMD:C_1206_3216Metric_Pad1.33x1.80mm_HandSolder, F.Cu at (156.5, 160.2)
- added C70: 22uF, Capacitor_SMD:C_1206_3216Metric_Pad1.33x1.80mm_HandSolder, F.Cu at (147.5, 32.3)
- added C71: 22uF, Capacitor_SMD:C_1206_3216Metric_Pad1.33x1.80mm_HandSolder, F.Cu at (231.8, 16.7)
- added C72: 22uF, Capacitor_SMD:C_1206_3216Metric_Pad1.33x1.80mm_HandSolder, F.Cu at (226.5, -7.43)
- added C73: 22uF, Capacitor_SMD:C_1206_3216Metric_Pad1.33x1.80mm_HandSolder, F.Cu at (226.5, -4.08)
- added C74: 22uF, Capacitor_SMD:C_1206_3216Metric_Pad1.33x1.80mm_HandSolder, F.Cu at (51.5, 82.3)
- added C75: 22uF, Capacitor_SMD:C_1206_3216Metric_Pad1.33x1.80mm_HandSolder, F.Cu at (185.9, 84.8)
- added C76: 22uF, Capacitor_SMD:C_1206_3216Metric_Pad1.33x1.80mm_HandSolder, F.Cu at (296.5, 85.8)
- added C77: 22uF, Capacitor_SMD:C_1206_3216Metric_Pad1.33x1.80mm_HandSolder, F.Cu at (132.0, 85.7)
- added C78: 22uF, Capacitor_SMD:C_1206_3216Metric_Pad1.33x1.80mm_HandSolder, F.Cu at (242.1, 85.9)
- added C79: 22uF, Capacitor_SMD:C_1206_3216Metric_Pad1.33x1.80mm_HandSolder, F.Cu at (347.6, 85.5)
- added C80: 1u, Capacitor_SMD:C_0603_1608Metric_Pad1.08x0.95mm_HandSolder, F.Cu at (60.0, 134.2)
- added C81: 10u, Capacitor_SMD:C_1206_3216Metric_Pad1.33x1.80mm_HandSolder, F.Cu at (52.1, 131.7)
- added C82: 100n, Capacitor_SMD:C_0603_1608Metric_Pad1.08x0.95mm_HandSolder, F.Cu at (54.0, 131.9)
- added C83: 15p, Capacitor_SMD:C_0603_1608Metric_Pad1.08x0.95mm_HandSolder, F.Cu at (61.7, 131.4)
- added C84: 15p, Capacitor_SMD:C_0603_1608Metric_Pad1.08x0.95mm_HandSolder, F.Cu at (61.7, 124.1)
- added C85: 100n, Capacitor_SMD:C_0603_1608Metric_Pad1.08x0.95mm_HandSolder, F.Cu at (149.8, 195.1)
- added D1: SD103AWS, Diode_SMD:D_SOD-323_HandSoldering, F.Cu at (51.1, 85.5)
- added D10: ESD5Zxx, Diode_SMD:D_SOD-523, F.Cu at (54.0, 124.3)
- added D2: SD103AWS, Diode_SMD:D_SOD-323_HandSoldering, F.Cu at (189.0, 85.2)
- added D3: SD103AWS, Diode_SMD:D_SOD-323_HandSoldering, F.Cu at (299.6, 86.2)
- added D4: SD103AWS, Diode_SMD:D_SOD-323_HandSoldering, F.Cu at (135.2, 86.1)
- added D5: SD103AWS, Diode_SMD:D_SOD-323_HandSoldering, F.Cu at (245.2, 86.3)
- added D6: SD103AWS, Diode_SMD:D_SOD-323_HandSoldering, F.Cu at (350.8, 86.0)
- added D7: SS34, Diode_SMD:D_SMA, F.Cu at (231.0, 12.4)
- added F1: 1.5A, Fuse:Fuse_1206_3216Metric, F.Cu at (57.6, 120.4)
- added IC6: TCA9617ADGKR, Eeloo_Pad:SOP65P490X110-8N, F.Cu at (162.9, -7.16)
- added IC7: SN74AHCT1G125DBVR, Eeloo_Pad:SOT95P280X145-5N, F.Cu at (147.6, 36.5)
- added J10: Conn_01x03_Pin, Connector_JST:JST_EH_B3B-EH-A_1x03_P2.50mm_Vertical, F.Cu at (285.9, 39.7)
- added J11: Conn_01x03_Pin, Connector_JST:JST_EH_B3B-EH-A_1x03_P2.50mm_Vertical, F.Cu at (291.8, 39.7)
- added J12: SC0914_13_, Eeloo_Pad:SC091413, F.Cu at (150.4, 144.2)
- added J13: SC0914_13_, Eeloo_Pad:SC091413, F.Cu at (216.9, -5.64)
- added J14: Conn_01x03_Pin, Connector_JST:JST_EH_B3B-EH-A_1x03_P2.50mm_Vertical, F.Cu at (297.6, 39.7)
- added J44: Conn_01x02_Pin, Connector_JST:JST_EH_B2B-EH-A_1x02_P2.50mm_Vertical, F.Cu at (229.9, 7.93)
- added J5: Conn_01x03_Pin, Connector_JST:JST_EH_B3B-EH-A_1x03_P2.50mm_Vertical, F.Cu at (262.5, 39.7)
- added J6: Conn_01x03_Pin, Connector_JST:JST_EH_B3B-EH-A_1x03_P2.50mm_Vertical, F.Cu at (268.4, 39.7)
- added J7: Conn_01x02_Pin, Connector_JST:JST_EH_B2B-EH-A_1x02_P2.50mm_Vertical, F.Cu at (262.5, 27.6)
- added J8: Conn_01x03_Pin, Connector_JST:JST_EH_B3B-EH-A_1x03_P2.50mm_Vertical, F.Cu at (274.2, 39.7)
- added J9: Conn_01x03_Pin, Connector_JST:JST_EH_B3B-EH-A_1x03_P2.50mm_Vertical, F.Cu at (280.1, 39.7)
- added L1: 3.9uH, Inductor_SMD:L_Sunlord_SWPA4030S, F.Cu at (84.0, 122.4)
- added LED37: FJ5241AH, Eeloo_Pad:LED-SEG-TH_18P-L25.2-W21.1-P2.54-LS15.2-BL, F.Cu at (344.7, 101.4)
- added Q1: AO3400A, Package_TO_SOT_SMD:SOT-23, F.Cu at (228.5, 16.1)
- added R100: 10k, Resistor_SMD:R_0603_1608Metric_Pad0.98x0.95mm_HandSolder, F.Cu at (323.1, 81.7)
- added R101: 10k, Resistor_SMD:R_0603_1608Metric_Pad0.98x0.95mm_HandSolder, F.Cu at (325.6, 81.7)
- added R102: 10k, Resistor_SMD:R_0603_1608Metric_Pad0.98x0.95mm_HandSolder, F.Cu at (328.1, 81.7)
- added R103: 10k, Resistor_SMD:R_0603_1608Metric_Pad0.98x0.95mm_HandSolder, F.Cu at (330.6, 81.7)
- added R104: 10k, Resistor_SMD:R_0603_1608Metric_Pad0.98x0.95mm_HandSolder, F.Cu at (333.1, 81.7)
- added R105: 4k7, Resistor_SMD:R_0603_1608Metric_Pad0.98x0.95mm_HandSolder, F.Cu at (161.2, -3.14)
- added R106: 4k7, Resistor_SMD:R_0603_1608Metric_Pad0.98x0.95mm_HandSolder, F.Cu at (161.2, -0.63)
- added R107: 10k, Resistor_SMD:R_0603_1608Metric_Pad0.98x0.95mm_HandSolder, F.Cu at (340.1, 54.2)
- added R108: 10k, Resistor_SMD:R_0603_1608Metric_Pad0.98x0.95mm_HandSolder, F.Cu at (320.0, 31.3)
- added R109: 10k, Resistor_SMD:R_0603_1608Metric_Pad0.98x0.95mm_HandSolder, F.Cu at (322.6, 31.3)
- added R11: 27.4, Resistor_SMD:R_0402_1005Metric_Pad0.72x0.64mm_HandSolder, F.Cu at (209.3, -14.4)
- added R110: 10k, Resistor_SMD:R_0603_1608Metric_Pad0.98x0.95mm_HandSolder, F.Cu at (325.1, 31.3)
- added R111: 10k, Resistor_SMD:R_0603_1608Metric_Pad0.98x0.95mm_HandSolder, F.Cu at (327.6, 31.3)
- added R112: 10k, Resistor_SMD:R_0603_1608Metric_Pad0.98x0.95mm_HandSolder, F.Cu at (330.1, 31.3)
- added R113: 10k, Resistor_SMD:R_0603_1608Metric_Pad0.98x0.95mm_HandSolder, F.Cu at (332.6, 31.3)
- added R114: 10k, Resistor_SMD:R_0603_1608Metric_Pad0.98x0.95mm_HandSolder, F.Cu at (335.1, 31.3)
- added R115: 10k, Resistor_SMD:R_0603_1608Metric_Pad0.98x0.95mm_HandSolder, F.Cu at (337.6, 31.3)
- added R116: 10k, Resistor_SMD:R_0603_1608Metric_Pad0.98x0.95mm_HandSolder, F.Cu at (340.1, 31.3)
- added R117: 10k, Resistor_SMD:R_0603_1608Metric_Pad0.98x0.95mm_HandSolder, F.Cu at (342.6, 31.3)
- added R118: 10k, Resistor_SMD:R_0603_1608Metric_Pad0.98x0.95mm_HandSolder, F.Cu at (345.1, 31.3)
- added R119: 10k, Resistor_SMD:R_0603_1608Metric_Pad0.98x0.95mm_HandSolder, F.Cu at (228.5, 19.0)
- added R12: 27.4, Resistor_SMD:R_0402_1005Metric_Pad0.72x0.64mm_HandSolder, F.Cu at (209.3, -11.9)
- added R120: 100, Resistor_SMD:R_0603_1608Metric_Pad0.98x0.95mm_HandSolder, F.Cu at (228.5, 20.5)
- added R121: 5.1k, Resistor_SMD:R_0603_1608Metric_Pad0.98x0.95mm_HandSolder, F.Cu at (44.3, 119.6)
- added R122: 5.1k, Resistor_SMD:R_0603_1608Metric_Pad0.98x0.95mm_HandSolder, F.Cu at (48.9, 138.0)
- added R123: 10k, Resistor_SMD:R_0603_1608Metric_Pad0.98x0.95mm_HandSolder, F.Cu at (56.6, 132.7)
- added R124: 10k, Resistor_SMD:R_0603_1608Metric_Pad0.98x0.95mm_HandSolder, F.Cu at (149.8, 197.6)
- added R125: 10k, Resistor_SMD:R_0603_1608Metric_Pad0.98x0.95mm_HandSolder, F.Cu at (149.8, 200.1)
- added R13: 39k, Resistor_SMD:R_0603_1608Metric_Pad0.98x0.95mm_HandSolder, F.Cu at (83.9, 79.8)
- added R14: 39k, Resistor_SMD:R_0603_1608Metric_Pad0.98x0.95mm_HandSolder, F.Cu at (86.5, 79.8)
- added R15: 39k, Resistor_SMD:R_0603_1608Metric_Pad0.98x0.95mm_HandSolder, F.Cu at (89.0, 79.8)
- added R16: 39k, Resistor_SMD:R_0603_1608Metric_Pad0.98x0.95mm_HandSolder, F.Cu at (166.5, 85.6)
- added R17: 39k, Resistor_SMD:R_0603_1608Metric_Pad0.98x0.95mm_HandSolder, F.Cu at (169.0, 85.6)
- added R18: 39k, Resistor_SMD:R_0603_1608Metric_Pad0.98x0.95mm_HandSolder, F.Cu at (171.5, 85.6)
- added R19: 39k, Resistor_SMD:R_0603_1608Metric_Pad0.98x0.95mm_HandSolder, F.Cu at (277.1, 86.6)
- added R20: 39k, Resistor_SMD:R_0603_1608Metric_Pad0.98x0.95mm_HandSolder, F.Cu at (279.6, 86.6)
- added R21: 39k, Resistor_SMD:R_0603_1608Metric_Pad0.98x0.95mm_HandSolder, F.Cu at (282.1, 86.6)
- added R22: 39k, Resistor_SMD:R_0603_1608Metric_Pad0.98x0.95mm_HandSolder, F.Cu at (112.6, 86.5)
- added R23: 39k, Resistor_SMD:R_0603_1608Metric_Pad0.98x0.95mm_HandSolder, F.Cu at (115.1, 86.5)
- added R24: 39k, Resistor_SMD:R_0603_1608Metric_Pad0.98x0.95mm_HandSolder, F.Cu at (117.7, 86.5)
- added R25: 39k, Resistor_SMD:R_0603_1608Metric_Pad0.98x0.95mm_HandSolder, F.Cu at (222.7, 86.7)
- added R26: 39k, Resistor_SMD:R_0603_1608Metric_Pad0.98x0.95mm_HandSolder, F.Cu at (225.2, 86.7)
- added R27: 39k, Resistor_SMD:R_0603_1608Metric_Pad0.98x0.95mm_HandSolder, F.Cu at (227.7, 86.7)
- added R28: 39k, Resistor_SMD:R_0603_1608Metric_Pad0.98x0.95mm_HandSolder, F.Cu at (328.2, 86.4)
- added R29: 39k, Resistor_SMD:R_0603_1608Metric_Pad0.98x0.95mm_HandSolder, F.Cu at (330.8, 86.4)
- added R30: 39k, Resistor_SMD:R_0603_1608Metric_Pad0.98x0.95mm_HandSolder, F.Cu at (333.3, 86.4)
- added R31: 10k, Resistor_SMD:R_0603_1608Metric_Pad0.98x0.95mm_HandSolder, F.Cu at (105.3, 56.3)
- added R32: 10k, Resistor_SMD:R_0603_1608Metric_Pad0.98x0.95mm_HandSolder, F.Cu at (107.9, 56.3)
- added R33: 10k, Resistor_SMD:R_0603_1608Metric_Pad0.98x0.95mm_HandSolder, F.Cu at (110.4, 56.3)
- added R34: 10k, Resistor_SMD:R_0603_1608Metric_Pad0.98x0.95mm_HandSolder, F.Cu at (112.9, 56.3)
- added R35: 10k, Resistor_SMD:R_0603_1608Metric_Pad0.98x0.95mm_HandSolder, F.Cu at (115.4, 56.3)
- added R36: 10k, Resistor_SMD:R_0603_1608Metric_Pad0.98x0.95mm_HandSolder, F.Cu at (117.9, 56.3)
- added R37: 10k, Resistor_SMD:R_0603_1608Metric_Pad0.98x0.95mm_HandSolder, F.Cu at (120.4, 56.3)
- added R38: 10k, Resistor_SMD:R_0603_1608Metric_Pad0.98x0.95mm_HandSolder, F.Cu at (122.9, 56.3)
- added R39: 10k, Resistor_SMD:R_0603_1608Metric_Pad0.98x0.95mm_HandSolder, F.Cu at (125.4, 56.3)
- added R40: 10k, Resistor_SMD:R_0603_1608Metric_Pad0.98x0.95mm_HandSolder, F.Cu at (127.9, 56.3)
- added R41: 10k, Resistor_SMD:R_0603_1608Metric_Pad0.98x0.95mm_HandSolder, F.Cu at (130.4, 56.3)
- added R42: 10k, Resistor_SMD:R_0603_1608Metric_Pad0.98x0.95mm_HandSolder, F.Cu at (133.0, 56.3)
- added R43: 10k, Resistor_SMD:R_0603_1608Metric_Pad0.98x0.95mm_HandSolder, F.Cu at (102.8, 51.9)
- added R44: 10k, Resistor_SMD:R_0603_1608Metric_Pad0.98x0.95mm_HandSolder, F.Cu at (105.3, 51.9)
- added R45: 10k, Resistor_SMD:R_0603_1608Metric_Pad0.98x0.95mm_HandSolder, F.Cu at (107.9, 51.9)
- added R46: 10k, Resistor_SMD:R_0603_1608Metric_Pad0.98x0.95mm_HandSolder, F.Cu at (110.4, 51.9)
- added R47: 10k, Resistor_SMD:R_0603_1608Metric_Pad0.98x0.95mm_HandSolder, F.Cu at (112.9, 51.9)
- added R48: 10k, Resistor_SMD:R_0603_1608Metric_Pad0.98x0.95mm_HandSolder, F.Cu at (115.4, 51.9)
- added R49: 10k, Resistor_SMD:R_0603_1608Metric_Pad0.98x0.95mm_HandSolder, F.Cu at (117.9, 51.9)
- added R50: 10k, Resistor_SMD:R_0603_1608Metric_Pad0.98x0.95mm_HandSolder, F.Cu at (120.4, 51.9)
- added R51: 10k, Resistor_SMD:R_0603_1608Metric_Pad0.98x0.95mm_HandSolder, F.Cu at (122.9, 51.9)
- added R52: 10k, Resistor_SMD:R_0603_1608Metric_Pad0.98x0.95mm_HandSolder, F.Cu at (125.4, 51.9)
- added R53: 10k, Resistor_SMD:R_0603_1608Metric_Pad0.98x0.95mm_HandSolder, F.Cu at (127.9, 51.9)
- added R54: 10k, Resistor_SMD:R_0603_1608Metric_Pad0.98x0.95mm_HandSolder, F.Cu at (130.4, 51.9)
- added R55: 10k, Resistor_SMD:R_0603_1608Metric_Pad0.98x0.95mm_HandSolder, F.Cu at (133.0, 51.9)
- added R56: 10k, Resistor_SMD:R_0603_1608Metric_Pad0.98x0.95mm_HandSolder, F.Cu at (102.8, 47.6)
- added R57: 10k, Resistor_SMD:R_0603_1608Metric_Pad0.98x0.95mm_HandSolder, F.Cu at (105.3, 47.6)
- added R58: 10k, Resistor_SMD:R_0603_1608Metric_Pad0.98x0.95mm_HandSolder, F.Cu at (107.9, 47.6)
- added R59: 10k, Resistor_SMD:R_0603_1608Metric_Pad0.98x0.95mm_HandSolder, F.Cu at (110.4, 47.6)
- added R60: 4k7, Resistor_SMD:R_0603_1608Metric_Pad0.98x0.95mm_HandSolder, F.Cu at (155.1, -8.64)
- added R61: 4k7, Resistor_SMD:R_0603_1608Metric_Pad0.98x0.95mm_HandSolder, F.Cu at (155.1, -6.13)
- added R62: 10k, Resistor_SMD:R_0603_1608Metric_Pad0.98x0.95mm_HandSolder, F.Cu at (155.1, -3.62)
- added R63: 4k7, Resistor_SMD:R_0603_1608Metric_Pad0.98x0.95mm_HandSolder, F.Cu at (155.1, -1.11)
- added R64: 4k7, Resistor_SMD:R_0603_1608Metric_Pad0.98x0.95mm_HandSolder, F.Cu at (155.1, 1.40)
- added R65: 10k, Resistor_SMD:R_0603_1608Metric_Pad0.98x0.95mm_HandSolder, F.Cu at (267.6, 53.2)
- added R66: 10k, Resistor_SMD:R_0603_1608Metric_Pad0.98x0.95mm_HandSolder, F.Cu at (264.2, 53.2)
- added R67: 10k, Resistor_SMD:R_0603_1608Metric_Pad0.98x0.95mm_HandSolder, F.Cu at (280.0, 55.6)
- added R68: 10k, Resistor_SMD:R_0603_1608Metric_Pad0.98x0.95mm_HandSolder, F.Cu at (282.5, 55.6)
- added R69: 10k, Resistor_SMD:R_0603_1608Metric_Pad0.98x0.95mm_HandSolder, F.Cu at (79.5, 84.0)
- added R70: 10k, Resistor_SMD:R_0603_1608Metric_Pad0.98x0.95mm_HandSolder, F.Cu at (55.9, 76.6)
- added R71: 10k, Resistor_SMD:R_0603_1608Metric_Pad0.98x0.95mm_HandSolder, F.Cu at (59.3, 80.0)
- added R72: 10k, Resistor_SMD:R_0603_1608Metric_Pad0.98x0.95mm_HandSolder, F.Cu at (59.3, 81.5)
- added R73: 10k, Resistor_SMD:R_0603_1608Metric_Pad0.98x0.95mm_HandSolder, F.Cu at (79.5, 85.5)
- added R74: 10k, Resistor_SMD:R_0603_1608Metric_Pad0.98x0.95mm_HandSolder, F.Cu at (55.9, 78.1)
- added R75: 10k, Resistor_SMD:R_0603_1608Metric_Pad0.98x0.95mm_HandSolder, F.Cu at (159.0, 80.3)
- added R76: 10k, Resistor_SMD:R_0603_1608Metric_Pad0.98x0.95mm_HandSolder, F.Cu at (161.5, 80.3)
- added R77: 10k, Resistor_SMD:R_0603_1608Metric_Pad0.98x0.95mm_HandSolder, F.Cu at (164.1, 80.3)
- added R78: 10k, Resistor_SMD:R_0603_1608Metric_Pad0.98x0.95mm_HandSolder, F.Cu at (166.6, 80.3)
- added R79: 10k, Resistor_SMD:R_0603_1608Metric_Pad0.98x0.95mm_HandSolder, F.Cu at (169.1, 80.3)
- added R80: 10k, Resistor_SMD:R_0603_1608Metric_Pad0.98x0.95mm_HandSolder, F.Cu at (171.6, 80.3)
- added R81: 10k, Resistor_SMD:R_0603_1608Metric_Pad0.98x0.95mm_HandSolder, F.Cu at (281.5, 82.4)
- added R82: 10k, Resistor_SMD:R_0603_1608Metric_Pad0.98x0.95mm_HandSolder, F.Cu at (265.5, 82.1)
- added R83: 10k, Resistor_SMD:R_0603_1608Metric_Pad0.98x0.95mm_HandSolder, F.Cu at (268.0, 82.1)
- added R84: 10k, Resistor_SMD:R_0603_1608Metric_Pad0.98x0.95mm_HandSolder, F.Cu at (270.5, 82.1)
- added R85: 10k, Resistor_SMD:R_0603_1608Metric_Pad0.98x0.95mm_HandSolder, F.Cu at (273.0, 82.1)
- added R86: 10k, Resistor_SMD:R_0603_1608Metric_Pad0.98x0.95mm_HandSolder, F.Cu at (275.5, 82.1)
- added R87: 10k, Resistor_SMD:R_0603_1608Metric_Pad0.98x0.95mm_HandSolder, F.Cu at (119.2, 76.2)
- added R88: 10k, Resistor_SMD:R_0603_1608Metric_Pad0.98x0.95mm_HandSolder, F.Cu at (121.7, 76.2)
- added R89: 10k, Resistor_SMD:R_0603_1608Metric_Pad0.98x0.95mm_HandSolder, F.Cu at (124.2, 76.2)
- added R90: 10k, Resistor_SMD:R_0603_1608Metric_Pad0.98x0.95mm_HandSolder, F.Cu at (126.7, 76.2)
- added R91: 10k, Resistor_SMD:R_0603_1608Metric_Pad0.98x0.95mm_HandSolder, F.Cu at (129.2, 76.2)
- added R92: 10k, Resistor_SMD:R_0603_1608Metric_Pad0.98x0.95mm_HandSolder, F.Cu at (131.7, 76.2)
- added R93: 10k, Resistor_SMD:R_0603_1608Metric_Pad0.98x0.95mm_HandSolder, F.Cu at (224.8, 81.4)
- added R94: 10k, Resistor_SMD:R_0603_1608Metric_Pad0.98x0.95mm_HandSolder, F.Cu at (227.3, 81.4)
- added R95: 10k, Resistor_SMD:R_0603_1608Metric_Pad0.98x0.95mm_HandSolder, F.Cu at (213.3, 81.5)
- added R96: 10k, Resistor_SMD:R_0603_1608Metric_Pad0.98x0.95mm_HandSolder, F.Cu at (215.8, 81.5)
- added R97: 10k, Resistor_SMD:R_0603_1608Metric_Pad0.98x0.95mm_HandSolder, F.Cu at (218.3, 81.5)
- added R98: 10k, Resistor_SMD:R_0603_1608Metric_Pad0.98x0.95mm_HandSolder, F.Cu at (220.8, 81.5)
- added R99: 10k, Resistor_SMD:R_0603_1608Metric_Pad0.98x0.95mm_HandSolder, F.Cu at (320.5, 81.7)
- added SW10: SW_Push, Button_Switch_SMD:SW_Push_1P1T_XKB_TS-1187A, F.Cu at (86.5, 57.6)
- added SW11: SW_Push, Button_Switch_SMD:SW_Push_1P1T_XKB_TS-1187A, F.Cu at (92.5, 57.6)
- added SW12: SW_Push, Button_Switch_SMD:SW_Push_1P1T_XKB_TS-1187A, F.Cu at (98.6, 57.6)
- added SW13: SW_Push, Button_Switch_SMD:SW_Push_1P1T_XKB_TS-1187A, F.Cu at (56.2, 47.3)
- added SW14: SW_Push, Button_Switch_SMD:SW_Push_1P1T_XKB_TS-1187A, F.Cu at (62.3, 47.3)
- added SW15: SW_Push, Button_Switch_SMD:SW_Push_1P1T_XKB_TS-1187A, F.Cu at (68.3, 47.3)
- added SW16: SW_Push, Button_Switch_SMD:SW_Push_1P1T_XKB_TS-1187A, F.Cu at (74.4, 47.3)
- added SW17: SW_Push, Button_Switch_SMD:SW_Push_1P1T_XKB_TS-1187A, F.Cu at (80.4, 47.3)
- added SW18: SW_Push, Button_Switch_SMD:SW_Push_1P1T_XKB_TS-1187A, F.Cu at (86.5, 47.3)
- added SW19: SW_Push, Button_Switch_SMD:SW_Push_1P1T_XKB_TS-1187A, F.Cu at (92.5, 47.3)
- added SW20: SW_Push, Button_Switch_SMD:SW_Push_1P1T_XKB_TS-1187A, F.Cu at (98.6, 47.3)
- added SW21: SW_Push, Button_Switch_SMD:SW_Push_1P1T_XKB_TS-1187A, F.Cu at (56.2, 36.9)
- added SW22: SW_Push, Button_Switch_SMD:SW_Push_1P1T_XKB_TS-1187A, F.Cu at (62.3, 36.9)
- added SW23: SW_Push, Button_Switch_SMD:SW_Push_1P1T_XKB_TS-1187A, F.Cu at (68.3, 36.9)
- added SW24: SW_Push, Button_Switch_SMD:SW_Push_1P1T_XKB_TS-1187A, F.Cu at (74.4, 36.9)
- added SW25: SW_Push, Button_Switch_SMD:SW_Push_1P1T_XKB_TS-1187A, F.Cu at (80.4, 36.9)
- added SW26: SW_Push, Button_Switch_SMD:SW_Push_1P1T_XKB_TS-1187A, F.Cu at (86.5, 36.9)
- added SW27: SW_Push, Button_Switch_SMD:SW_Push_1P1T_XKB_TS-1187A, F.Cu at (92.5, 36.9)
- added SW28: SW_Push, Button_Switch_SMD:SW_Push_1P1T_XKB_TS-1187A, F.Cu at (98.6, 36.9)
- added SW29: SW_Push, Button_Switch_SMD:SW_Push_1P1T_XKB_TS-1187A, F.Cu at (56.2, 26.6)
- added SW30: SW_Push, Button_Switch_SMD:SW_Push_1P1T_XKB_TS-1187A, F.Cu at (62.3, 26.6)
- added SW31: SW_Push, Button_Switch_SMD:SW_Push_1P1T_XKB_TS-1187A, F.Cu at (68.3, 26.6)
- added SW32: SW_Push, Button_Switch_SMD:SW_Push_1P1T_XKB_TS-1187A, F.Cu at (74.4, 26.6)
- added SW33: SW_Push, Button_Switch_SMD:SW_Push_1P1T_XKB_TS-1187A, F.Cu at (80.4, 26.6)
- added SW5: SW_Push, Button_Switch_SMD:SW_Push_1P1T_XKB_TS-1187A, F.Cu at (56.2, 57.6)
- added SW6: SW_Push, Button_Switch_SMD:SW_Push_1P1T_XKB_TS-1187A, F.Cu at (62.3, 57.6)
- added SW7: SW_Push, Button_Switch_SMD:SW_Push_1P1T_XKB_TS-1187A, F.Cu at (68.3, 57.6)
- added SW8: SW_Push, Button_Switch_SMD:SW_Push_1P1T_XKB_TS-1187A, F.Cu at (74.4, 57.6)
- added SW9: SW_Push, Button_Switch_SMD:SW_Push_1P1T_XKB_TS-1187A, F.Cu at (80.4, 57.6)
- added U7: AP63203WU, Package_TO_SOT_SMD:TSOT-23-6, F.Cu at (81.9, 124.9)
- added U8: CH334F, Package_DFN_QFN:QFN-24-1EP_4x4mm_P0.5mm_EP2.7x2.7mm, F.Cu at (56.5, 127.9)
- added U9: USBLC6-2SC6, Package_TO_SOT_SMD:SOT-23-6, F.Cu at (65.6, 120.9)
- added Y3: 12MHz, Crystal:Crystal_SMD_3225-4Pin_3.2x2.5mm_HandSoldering, F.Cu at (62.0, 127.8)
- C15, C30: footprint Capacitor_SMD:C_0603_1608Metric_Pad1.08x0.95mm_HandSolder -> Capacitor_SMD:C_1206_3216Metric_Pad1.33x1.80mm_HandSolder
- IC2: value W25Q16JVUXIQ_TR -> PCA9535PW; footprint Eeloo_Pad:SON50P300X200X60-9N -> Package_SO:TSSOP-24_4.4x7.8mm_P0.65mm
- IC3: value ADS1015IDGST -> PCA9535PW; footprint Eeloo_Pad:SOP50P490X110-10N -> Package_SO:TSSOP-24_4.4x7.8mm_P0.65mm
- IC4: value PCF8575DBQR -> ADS7830IPWR; footprint Eeloo_Pad:SOP64P600X175-24N -> Eeloo_Pad:SOP65P640X120-16N
- IC5: value PCF8575DBQR -> W25Q16JVUXIQ_TR; footprint Eeloo_Pad:SOP64P600X175-24N -> Eeloo_Pad:SON50P300X200X60-9N
- J2: footprint Connector_JST:JST_GH_SM12B-GHS-TB_1x12-1MP_P1.25mm_Horizontal -> Connector_JST:JST_GH_SM13B-GHS-TB_1x13-1MP_P1.25mm_Horizontal
- J3: value SC0914_13_ -> Conn_01x02_Pin; footprint Eeloo_Pad:SC091413 -> Connector_JST:JST_EH_B2B-EH-A_1x02_P2.50mm_Vertical
- J4: value SC0914_13_ -> Conn_01x03_Pin; footprint Eeloo_Pad:SC091413 -> Connector_JST:JST_EH_B3B-EH-A_1x03_P2.50mm_Vertical
- LED1, LED10, LED11, LED12, LED2, LED3, LED4, LED5, LED6, LED7, LED8, LED9: value FJ5241AH -> XL-5050RGBC-WS2812B; footprint Eeloo_Pad:LED-SEG-TH_18P-L25.2-W21.1-P2.54-LS15.2-BL -> Eeloo_Pad:LED-SMD_4P-L5.0-W5.0-BL_XL-5050RGBC
- LED26, LED27, LED28, LED29, LED30, LED31, LED32, LED33, LED34, LED35, LED36: value XL-5050RGBC-WS2812B -> FJ5241AH; footprint Eeloo_Pad:LED-SMD_4P-L5.0-W5.0-BL_XL-5050RGBC -> Eeloo_Pad:LED-SEG-TH_18P-L25.2-W21.1-P2.54-LS15.2-BL
- R1: value 1k -> 10k
- R10, R5: value 27.2 -> 1k
- R2: value NC -> 10k
- R4, R9: value 27.2 -> NC
- R6: value 1k -> 27.4; footprint Resistor_SMD:R_0603_1608Metric_Pad0.98x0.95mm_HandSolder -> Resistor_SMD:R_0402_1005Metric_Pad0.72x0.64mm_HandSolder
- R7: value NC -> 27.4; footprint Resistor_SMD:R_0603_1608Metric_Pad0.98x0.95mm_HandSolder -> Resistor_SMD:R_0402_1005Metric_Pad0.72x0.64mm_HandSolder
- SW1, SW2, SW3, SW4: footprint Button_Switch_SMD:SW_SPST_TL3305A -> Button_Switch_SMD:SW_Push_1P1T_XKB_TS-1187A
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Connections:
- C1 pad 1: /navball_module/+3.3V -> +3.3V
- C10 pad 1: /navball_module/+3.3V -> +3.3V
- C11 pad 1: /navball_module/+3.3V -> +3.3V
- C12 pad 1: /navball_module/+3.3V -> +3.3V
- C13 pad 1: /navball_module/+3.3V -> +3.3V
- C14 pad 1: /navball_module/+3.3V -> +3.3V
- C15 pad 1: /navball_module/+3.3V -> +3.3V
- C16 pad 1: /control_module/+3.3V -> +3.3V
- C22 pad 1: /control_module/+3.3V -> +3.3V
- C23 pad 1: /control_module/+3.3V -> +3.3V
- C24 pad 1: /control_module/+3.3V -> +3.3V
- C25 pad 1: /control_module/+3.3V -> +3.3V
- C26 pad 1: /control_module/+3.3V -> +3.3V
- C27 pad 1: /control_module/+3.3V -> +3.3V
- C28 pad 1: /control_module/+3.3V -> +3.3V
- C29 pad 1: /control_module/+3.3V -> +3.3V
- C30 pad 1: /control_module/+3.3V -> +3.3V
- C31 pad 1: /navball_module/+3.3V -> +3.3V
- C32 pad 1: /navball_module/+3.3V -> +3.3V
- C33 pad 1: /navball_module/+3.3V -> +3.3V
- C7 pad 1: /navball_module/+3.3V -> +3.3V
- C8 pad 1: /navball_module/+3.3V -> +3.3V
- C9 pad 1: /navball_module/+3.3V -> +3.3V
- IC1 pad 8: /navball_module/+3.3V -> +3.3V
- IC2 pad 1: /control_module/uC1/QSPI_SS -> /control_module/I2C_GPIO_EXT0_INT
- IC2 pad 2: /control_module/uC1/QSPI_SD1 -> Net-(IC2-A1)
- IC2 pad 3: /control_module/uC1/QSPI_SD2 -> Net-(IC2-A2)
- IC2 pad 4: GND -> /control_module/SAS
- IC2 pad 5: /control_module/uC1/QSPI_SD0 -> /control_module/RCS
- IC2 pad 6: /control_module/uC1/QSPI_SCLK -> /control_module/CTRL0
- IC2 pad 7: /control_module/uC1/QSPI_SD3 -> /control_module/CTRL1
- IC2 pad 8: /control_module/+3.3V -> /control_module/CTRL2
- IC2 pad 9: GND -> /control_module/CTRL3
- IC3 pad 1: unconnected-(IC3-ADDR-Pad1) -> /control_module/I2C_GPIO_EXT1_INT
- IC3 pad 10: unconnected-(IC3-SCL-Pad10) -> /control_module/TARGET
- IC3 pad 2: unconnected-(IC3-ALERT/RDY-Pad2) -> Net-(IC3-A1)
- IC3 pad 3: unconnected-(IC3-GND-Pad3) -> Net-(IC3-A2)
- IC3 pad 4: unconnected-(IC3-AIN0-Pad4) -> /control_module/PROGRADE
- IC3 pad 5: unconnected-(IC3-AIN1-Pad5) -> /control_module/RETROGRADE
- IC3 pad 6: unconnected-(IC3-AIN2-Pad6) -> /control_module/NORMAL
- IC3 pad 7: unconnected-(IC3-AIN3-Pad7) -> /control_module/ANTINORMAL
- IC3 pad 8: unconnected-(IC3-VDD-Pad8) -> /control_module/RADIAL_IN
- IC3 pad 9: unconnected-(IC3-SDA-Pad9) -> /control_module/RADIAL_OUT
- IC4 pad 1: unconnected-(IC4-~{INT}-Pad1) -> /control_module/EXT1
- IC4 pad 10: unconnected-(IC4-P06-Pad10) -> +3.3V
- IC4 pad 11: unconnected-(IC4-P07-Pad11) -> GND
- IC4 pad 12: unconnected-(IC4-GND-Pad12) -> Net-(IC4-A0)
- IC4 pad 13: unconnected-(IC4-P10-Pad13) -> Net-(IC4-A1)
- IC4 pad 14: unconnected-(IC4-P11-Pad14) -> /control_module/I2C0_SCL_33
- IC4 pad 15: unconnected-(IC4-P12-Pad15) -> /control_module/I2C0_SDA_33
- IC4 pad 16: unconnected-(IC4-P13-Pad16) -> +3.3V
- IC4 pad 2: unconnected-(IC4-A1-Pad2) -> /control_module/THROTTLE
- IC4 pad 3: unconnected-(IC4-A2-Pad3) -> /control_module/JOY_D_AXIS_R
- IC4 pad 4: unconnected-(IC4-P00-Pad4) -> /control_module/JOY_D_AXIS_Y
- IC4 pad 5: unconnected-(IC4-P01-Pad5) -> /control_module/JOY_D_AXIS_X
- IC4 pad 6: unconnected-(IC4-P02-Pad6) -> /control_module/JOY_G_AXIS_R
- IC4 pad 7: unconnected-(IC4-P03-Pad7) -> /control_module/JOY_G_AXIS_Y
- IC4 pad 8: unconnected-(IC4-P04-Pad8) -> /control_module/JOY_G_AXIS_X
- IC4 pad 9: unconnected-(IC4-P05-Pad9) -> GND
- IC5 pad 1: unconnected-(IC5-~{INT}-Pad1) -> /control_module/uC1/QSPI_SS
- IC5 pad 2: unconnected-(IC5-A1-Pad2) -> /control_module/uC1/QSPI_SD1
- IC5 pad 3: unconnected-(IC5-A2-Pad3) -> /control_module/uC1/QSPI_SD2
- IC5 pad 4: unconnected-(IC5-P00-Pad4) -> GND
- IC5 pad 5: unconnected-(IC5-P01-Pad5) -> /control_module/uC1/QSPI_SD0
- IC5 pad 6: unconnected-(IC5-P02-Pad6) -> /control_module/uC1/QSPI_SCLK
- IC5 pad 7: unconnected-(IC5-P03-Pad7) -> /control_module/uC1/QSPI_SD3
- IC5 pad 8: unconnected-(IC5-P04-Pad8) -> +3.3V
- IC5 pad 9: unconnected-(IC5-P05-Pad9) -> GND
- J1 pad A1: Net-(J1-GND-PadA1) -> GND
- J1 pad A12: Net-(J1-GND-PadA1) -> GND
- J1 pad A4: /VBUS -> Net-(F1-Pad1)
- J1 pad A5: unconnected-(J1-CC1-PadA5) -> /CC1
- J1 pad A6: unconnected-(J1-D+-PadA6) -> /USB_DP
- J1 pad A7: unconnected-(J1-D--PadA7) -> /USB_DM
- J1 pad A9: /VBUS -> Net-(F1-Pad1)
- J1 pad B1: Net-(J1-GND-PadA1) -> GND
- J1 pad B12: Net-(J1-GND-PadA1) -> GND
- J1 pad B4: /VBUS -> Net-(F1-Pad1)
- J1 pad B5: unconnected-(J1-CC2-PadB5) -> /CC2
- J1 pad B6: unconnected-(J1-D+-PadB6) -> /USB_DP
- J1 pad B7: unconnected-(J1-D--PadB7) -> /USB_DM
- J1 pad B9: /VBUS -> Net-(F1-Pad1)
- J1 pad S1: unconnected-(J1-SHIELD-PadS1) -> GND
- J2 pad 1: /navball_module/+3.3V -> +3.3V
- J3 pad 1: /navball_module/+3.3V -> /control_module/JOY_BTN_G
- J3 pad 2: /navball_module/uC1/GPIO0 -> GND
- J4 pad 1: /control_module/+3.3V -> +3.3V
- J4 pad 2: /control_module/uC1/GPIO0 -> /control_module/JOY_G_AXIS_X
- J4 pad 3: /control_module/uC1/GPIO1 -> GND
- LED1 pad 1: /control_module/seg_4x14_module1/E -> /VBUS
- LED1 pad 2: /control_module/seg_4x14_module1/N -> Net-(LED1-DOU)
- LED1 pad 4: /control_module/seg_4x14_module1/M -> /control_module/LED_CTRL_50
- LED10 pad 1: /control_module/seg_4x14_module3/E -> /VBUS
- LED10 pad 2: /control_module/seg_4x14_module3/N -> Net-(LED10-DOU)
- LED10 pad 4: /control_module/seg_4x14_module3/M -> Net-(LED10-DIN)
- LED11 pad 1: /control_module/seg_4x14_module4/E -> /VBUS
- LED11 pad 2: /control_module/seg_4x14_module4/N -> Net-(LED11-DOU)
- LED11 pad 4: /control_module/seg_4x14_module4/M -> Net-(LED11-DIN)
- LED12 pad 1: /control_module/seg_4x14_module5/E -> /VBUS
- LED12 pad 2: /control_module/seg_4x14_module5/N -> Net-(LED12-DOU)
- LED12 pad 4: /control_module/seg_4x14_module5/M -> Net-(LED12-DIN)
- LED13 pad 1: unconnected-(LED13-VDD-Pad1) -> /VBUS
- LED13 pad 2: unconnected-(LED13-DOU-Pad2) -> Net-(LED13-DOU)
- LED13 pad 3: unconnected-(LED13-GND-Pad3) -> GND
- LED13 pad 4: unconnected-(LED13-DIN-Pad4) -> Net-(LED13-DIN)
- LED14 pad 1: unconnected-(LED14-VDD-Pad1) -> /VBUS
- LED14 pad 2: unconnected-(LED14-DOU-Pad2) -> Net-(LED14-DOU)
- LED14 pad 3: unconnected-(LED14-GND-Pad3) -> GND
- LED14 pad 4: unconnected-(LED14-DIN-Pad4) -> Net-(LED14-DIN)
- LED15 pad 1: unconnected-(LED15-VDD-Pad1) -> /VBUS
- LED15 pad 2: unconnected-(LED15-DOU-Pad2) -> Net-(LED15-DOU)
- LED15 pad 3: unconnected-(LED15-GND-Pad3) -> GND
- LED15 pad 4: unconnected-(LED15-DIN-Pad4) -> Net-(LED10-DOU)
- LED16 pad 1: unconnected-(LED16-VDD-Pad1) -> /VBUS
- LED16 pad 2: unconnected-(LED16-DOU-Pad2) -> Net-(LED16-DOU)
- LED16 pad 3: unconnected-(LED16-GND-Pad3) -> GND
- LED16 pad 4: unconnected-(LED16-DIN-Pad4) -> Net-(LED11-DOU)
- LED17 pad 1: unconnected-(LED17-VDD-Pad1) -> /VBUS
- LED17 pad 2: unconnected-(LED17-DOU-Pad2) -> Net-(LED17-DOU)
- LED17 pad 3: unconnected-(LED17-GND-Pad3) -> GND
- LED17 pad 4: unconnected-(LED17-DIN-Pad4) -> Net-(LED12-DOU)
- LED18 pad 1: unconnected-(LED18-VDD-Pad1) -> /VBUS
- LED18 pad 2: unconnected-(LED18-DOU-Pad2) -> Net-(LED18-DOU)
- LED18 pad 3: unconnected-(LED18-GND-Pad3) -> GND
- LED18 pad 4: unconnected-(LED18-DIN-Pad4) -> Net-(LED13-DOU)
- LED19 pad 1: unconnected-(LED19-VDD-Pad1) -> /VBUS
- LED19 pad 2: unconnected-(LED19-DOU-Pad2) -> Net-(LED19-DOU)
- LED19 pad 3: unconnected-(LED19-GND-Pad3) -> GND
- LED19 pad 4: unconnected-(LED19-DIN-Pad4) -> Net-(LED14-DOU)
- LED2 pad 1: /control_module/seg_4x14_module/E -> /VBUS
- LED2 pad 2: /control_module/seg_4x14_module/N -> Net-(LED2-DOU)
- LED2 pad 4: /control_module/seg_4x14_module/M -> Net-(LED2-DIN)
- LED20 pad 1: unconnected-(LED20-VDD-Pad1) -> /VBUS
- LED20 pad 2: unconnected-(LED20-DOU-Pad2) -> Net-(LED20-DOU)
- LED20 pad 3: unconnected-(LED20-GND-Pad3) -> GND
- LED20 pad 4: unconnected-(LED20-DIN-Pad4) -> Net-(LED15-DOU)
- LED21 pad 1: unconnected-(LED21-VDD-Pad1) -> /VBUS
- LED21 pad 2: unconnected-(LED21-DOU-Pad2) -> Net-(LED2-DIN)
- LED21 pad 3: unconnected-(LED21-GND-Pad3) -> GND
- LED21 pad 4: unconnected-(LED21-DIN-Pad4) -> Net-(LED16-DOU)
- LED22 pad 1: unconnected-(LED22-VDD-Pad1) -> /VBUS
- LED22 pad 2: unconnected-(LED22-DOU-Pad2) -> Net-(LED22-DOU)
- LED22 pad 3: unconnected-(LED22-GND-Pad3) -> GND
- LED22 pad 4: unconnected-(LED22-DIN-Pad4) -> Net-(LED17-DOU)
- LED23 pad 1: unconnected-(LED23-VDD-Pad1) -> /VBUS
- LED23 pad 2: unconnected-(LED23-DOU-Pad2) -> Net-(LED23-DOU)
- LED23 pad 3: unconnected-(LED23-GND-Pad3) -> GND
- LED23 pad 4: unconnected-(LED23-DIN-Pad4) -> Net-(LED18-DOU)
- LED24 pad 1: unconnected-(LED24-VDD-Pad1) -> /VBUS
- LED24 pad 2: unconnected-(LED24-DOU-Pad2) -> Net-(LED24-DOU)
- LED24 pad 3: unconnected-(LED24-GND-Pad3) -> GND
- LED24 pad 4: unconnected-(LED24-DIN-Pad4) -> Net-(LED19-DOU)
- LED25 pad 1: unconnected-(LED25-VDD-Pad1) -> /VBUS
- LED25 pad 3: unconnected-(LED25-GND-Pad3) -> GND
- LED25 pad 4: unconnected-(LED25-DIN-Pad4) -> Net-(LED20-DOU)
- LED26 pad 1: unconnected-(LED26-VDD-Pad1) -> /control_module/seg_4x14_module/E
- LED26 pad 2: unconnected-(LED26-DOU-Pad2) -> /control_module/seg_4x14_module/N
- LED26 pad 4: unconnected-(LED26-DIN-Pad4) -> /control_module/seg_4x14_module/M
- LED27 pad 1: unconnected-(LED27-VDD-Pad1) -> /control_module/seg_4x14_module/E
- LED27 pad 2: unconnected-(LED27-DOU-Pad2) -> /control_module/seg_4x14_module/N
- LED27 pad 4: unconnected-(LED27-DIN-Pad4) -> /control_module/seg_4x14_module/M
- LED28 pad 1: unconnected-(LED28-VDD-Pad1) -> /control_module/seg_4x14_module3/E
- LED28 pad 2: unconnected-(LED28-DOU-Pad2) -> /control_module/seg_4x14_module3/N
- LED28 pad 4: unconnected-(LED28-DIN-Pad4) -> /control_module/seg_4x14_module3/M
- LED29 pad 1: unconnected-(LED29-VDD-Pad1) -> /control_module/seg_4x14_module3/E
- LED29 pad 2: unconnected-(LED29-DOU-Pad2) -> /control_module/seg_4x14_module3/N
- LED29 pad 4: unconnected-(LED29-DIN-Pad4) -> /control_module/seg_4x14_module3/M
- LED3 pad 1: /control_module/seg_4x14_module2/E -> /VBUS
- LED3 pad 2: /control_module/seg_4x14_module2/N -> Net-(LED3-DOU)
- LED3 pad 4: /control_module/seg_4x14_module2/M -> Net-(LED22-DOU)
- LED30 pad 1: unconnected-(LED30-VDD-Pad1) -> /control_module/seg_4x14_module4/E
- LED30 pad 2: unconnected-(LED30-DOU-Pad2) -> /control_module/seg_4x14_module4/N
- LED30 pad 4: unconnected-(LED30-DIN-Pad4) -> /control_module/seg_4x14_module4/M
- LED31 pad 1: unconnected-(LED31-VDD-Pad1) -> /control_module/seg_4x14_module4/E
- LED31 pad 2: unconnected-(LED31-DOU-Pad2) -> /control_module/seg_4x14_module4/N
- LED31 pad 4: unconnected-(LED31-DIN-Pad4) -> /control_module/seg_4x14_module4/M
- LED32 pad 1: unconnected-(LED32-VDD-Pad1) -> /control_module/seg_4x14_module1/E
- LED32 pad 2: unconnected-(LED32-DOU-Pad2) -> /control_module/seg_4x14_module1/N
- LED32 pad 4: unconnected-(LED32-DIN-Pad4) -> /control_module/seg_4x14_module1/M
- LED33 pad 1: unconnected-(LED33-VDD-Pad1) -> /control_module/seg_4x14_module1/E
- LED33 pad 2: unconnected-(LED33-DOU-Pad2) -> /control_module/seg_4x14_module1/N
- LED33 pad 4: unconnected-(LED33-DIN-Pad4) -> /control_module/seg_4x14_module1/M
- LED34 pad 1: unconnected-(LED34-VDD-Pad1) -> /control_module/seg_4x14_module2/E
- LED34 pad 2: unconnected-(LED34-DOU-Pad2) -> /control_module/seg_4x14_module2/N
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Routing:
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Other:
- board text added: "JoY D"
- board text added: "JoY G"
- board text added: "NAV"
- board text added: "Stage"

Commit message: working on the routing of the pcb
Parts:
- removed R100, R101, R102, R103, R104, R69, R70, R71, R72, R73, R74, R75, R76, R77, R78, R79, R80, R81, R82, R83, R84, R85, R86, R87, R88, R89, R90, R91, R92, R93, R94, R95, R96, R97, R98, R99: 10k, Resistor_SMD:R_0603_1608Metric_Pad0.98x0.95mm_HandSolder
- added C100: 100n, Capacitor_SMD:C_0603_1608Metric_Pad1.08x0.95mm_HandSolder, F.Cu at (162.7, 8.13)
- added C101: 100n, Capacitor_SMD:C_0603_1608Metric_Pad1.08x0.95mm_HandSolder, F.Cu at (162.7, 10.6)
- added C102: 100n, Capacitor_SMD:C_0603_1608Metric_Pad1.08x0.95mm_HandSolder, F.Cu at (162.7, 13.1)
- added C103: 100n, Capacitor_SMD:C_0603_1608Metric_Pad1.08x0.95mm_HandSolder, F.Cu at (162.7, 15.7)
- added C104: 100n, Capacitor_SMD:C_0603_1608Metric_Pad1.08x0.95mm_HandSolder, F.Cu at (162.7, 18.2)
- added C105: 100n, Capacitor_SMD:C_0603_1608Metric_Pad1.08x0.95mm_HandSolder, F.Cu at (162.7, 20.7)
- added C106: 100n, Capacitor_SMD:C_0603_1608Metric_Pad1.08x0.95mm_HandSolder, F.Cu at (162.7, 23.2)
- added C107: 100n, Capacitor_SMD:C_0603_1608Metric_Pad1.08x0.95mm_HandSolder, F.Cu at (167.0, 8.13)
- added C108: 100n, Capacitor_SMD:C_0603_1608Metric_Pad1.08x0.95mm_HandSolder, F.Cu at (167.0, 10.6)
- added C109: 100n, Capacitor_SMD:C_0603_1608Metric_Pad1.08x0.95mm_HandSolder, F.Cu at (167.0, 13.1)
- added C110: 100n, Capacitor_SMD:C_0603_1608Metric_Pad1.08x0.95mm_HandSolder, F.Cu at (167.0, 15.7)
- added C86: 100n, Capacitor_SMD:C_0603_1608Metric_Pad1.08x0.95mm_HandSolder, F.Cu at (154.0, 8.13)
- added C87: 100n, Capacitor_SMD:C_0603_1608Metric_Pad1.08x0.95mm_HandSolder, F.Cu at (154.0, 10.6)
- added C88: 100n, Capacitor_SMD:C_0603_1608Metric_Pad1.08x0.95mm_HandSolder, F.Cu at (154.0, 13.1)
- added C89: 100n, Capacitor_SMD:C_0603_1608Metric_Pad1.08x0.95mm_HandSolder, F.Cu at (154.0, 15.7)
- added C90: 100n, Capacitor_SMD:C_0603_1608Metric_Pad1.08x0.95mm_HandSolder, F.Cu at (154.0, 18.2)
- added C91: 100n, Capacitor_SMD:C_0603_1608Metric_Pad1.08x0.95mm_HandSolder, F.Cu at (154.0, 20.7)
- added C92: 100n, Capacitor_SMD:C_0603_1608Metric_Pad1.08x0.95mm_HandSolder, F.Cu at (154.0, 23.2)
- added C93: 100n, Capacitor_SMD:C_0603_1608Metric_Pad1.08x0.95mm_HandSolder, F.Cu at (158.3, 8.13)
- added C94: 100n, Capacitor_SMD:C_0603_1608Metric_Pad1.08x0.95mm_HandSolder, F.Cu at (158.3, 10.6)
- added C95: 100n, Capacitor_SMD:C_0603_1608Metric_Pad1.08x0.95mm_HandSolder, F.Cu at (158.3, 13.1)
- added C96: 100n, Capacitor_SMD:C_0603_1608Metric_Pad1.08x0.95mm_HandSolder, F.Cu at (158.3, 15.7)
- added C97: 100n, Capacitor_SMD:C_0603_1608Metric_Pad1.08x0.95mm_HandSolder, F.Cu at (158.3, 18.2)
- added C98: 100n, Capacitor_SMD:C_0603_1608Metric_Pad1.08x0.95mm_HandSolder, F.Cu at (158.3, 20.7)
- added C99: 100n, Capacitor_SMD:C_0603_1608Metric_Pad1.08x0.95mm_HandSolder, F.Cu at (158.3, 23.2)
- added R126: 330, Resistor_SMD:R_0603_1608Metric_Pad0.98x0.95mm_HandSolder, F.Cu at (167.0, 18.2)
- added R127: 10k, Resistor_SMD:R_0603_1608Metric_Pad0.98x0.95mm_HandSolder, F.Cu at (167.0, 20.7)
- added R128: 10k, Resistor_SMD:R_0603_1608Metric_Pad0.98x0.95mm_HandSolder, F.Cu at (173.4, 8.13)
- added R129: 10k, Resistor_SMD:R_0603_1608Metric_Pad0.98x0.95mm_HandSolder, F.Cu at (173.4, 10.6)
- C46, C47, C48, C49, C50, C51, C52, C53, C54, C55, C56, C57, C74, C75, C76, C77, C78, C79, D1, D2, D3, D4, D5, D6, R13, R14, R15, R16, R17, R18, R19, R20, R21, R22, R23, R24, R25, R26, R27, R28, R29, R30, U1, U2, U3, U4, U5, U6: moved to B.Cu
- LED1, LED10, LED11, LED12, LED13, LED14, LED15, LED16, LED17, LED18, LED19, LED2, LED20, LED21, LED22, LED23, LED24, LED25, LED3, LED4, LED5, LED6, LED7, LED8, LED9: footprint Eeloo_Pad:LED-SMD_4P-L5.0-W5.0-BL_XL-5050RGBC -> LED_SMD:LED_WS2812B_PLCC4_5.0x5.0mm_P3.2mm
- Y3: footprint Crystal:Crystal_SMD_3225-4Pin_3.2x2.5mm_HandSoldering -> Eeloo_Pad:ABM8272T3
- moved R125 233.0 mm to (320.4, 41.3)
- moved R124 225.6 mm to (320.4, 49.8)
- moved C85 182.6 mm to (260.9, 50.2)
- moved R15 116.6 mm to (-25.7, 100.9), turned to 0 degrees
- moved R14 114.4 mm to (-25.7, 102.4), turned to 0 degrees
- moved R13 112.3 mm to (-25.7, 103.9), turned to 0 degrees
- moved LED26 96.9 mm to (-40.7, 102.4)
- moved LED27 96.9 mm to (-15.4, 102.4)
- moved C52 89.5 mm to (-5.18, 102.5), turned to -90 degrees
- moved C46 89.2 mm to (-8.59, 97.3), turned to 0 degrees
- moved U1 85.3 mm to (-13.7, 102.0)
- moved D1 76.1 mm to (-23.1, 102.6), turned to 90 degrees
- moved C74 62.1 mm to (-7.16, 102.5), turned to -90 degrees
- moved C53 39.8 mm to (200.4, 101.8), turned to -90 degrees
- moved C47 37.2 mm to (197.0, 96.5), turned to 0 degrees
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Connections:
- LED1 pad 4: /control_module/LED_CTRL_50 -> Net-(LED1-DIN)
- U8 pad 1: unconnected-(U8-~{OVCUR}-Pad1) -> /HUB_OVCUR
- U8 pad 18: unconnected-(U8-PSELF-Pad18) -> /HUB_PSELF
Routing:
- net /VBUS: track 29.9 -> 143.7 mm
- net GND: track 40.8 -> 108.1 mm, vias 0 -> 37
- net /control_module/seg_4x14_module4/AD: track 0.00 -> 47.3 mm, vias 0 -> 2
- net /control_module/seg_4x14_module1/AD: track 0.00 -> 47.3 mm, vias 0 -> 2
- net /control_module/seg_4x14_module3/AD: track 0.00 -> 47.3 mm, vias 0 -> 2
- net /control_module/seg_4x14_module/AD: track 0.00 -> 47.3 mm, vias 0 -> 2
- net /control_module/seg_4x14_module2/AD: track 0.00 -> 47.3 mm, vias 0 -> 2
- net /control_module/seg_4x14_module5/AD: track 0.00 -> 47.3 mm, vias 0 -> 2
- net /control_module/seg_4x14_module1/F: track 0.00 -> 45.9 mm
- net /control_module/seg_4x14_module2/F: track 0.00 -> 45.9 mm
- net /control_module/seg_4x14_module/F: track 0.00 -> 45.9 mm
- net /control_module/seg_4x14_module5/F: track 0.00 -> 45.9 mm
- net /control_module/seg_4x14_module3/F: track 0.00 -> 45.9 mm
- net /control_module/seg_4x14_module4/F: track 0.00 -> 45.9 mm
- net /control_module/seg_4x14_module4/E: track 0.00 -> 45.2 mm
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