File: Kicad/Eeloo_Pad.kicad_sch (KiCad schematic)
At the start: 1 part, among them J1 USB_C_Receptacle_USB2.0_16P

Commit message: schematics correction
Parts:
- added C58, C59, C60, C65, C66, C67, C68: 22uF, Capacitor_SMD:C_1206_3216Metric_Pad1.33x1.80mm_HandSolder, symbol Device:C
- added C61, C62, C63: 100nF, Capacitor_SMD:C_0603_1608Metric_Pad1.08x0.95mm_HandSolder, symbol Device:C
- added C64, C82: 100n, Capacitor_SMD:C_0603_1608Metric_Pad1.08x0.95mm_HandSolder, symbol Device:C
- added C80: 1u, Capacitor_SMD:C_0603_1608Metric_Pad1.08x0.95mm_HandSolder, symbol Device:C
- added C81: 10u, Capacitor_SMD:C_1206_3216Metric_Pad1.33x1.80mm_HandSolder, symbol Device:C
- added C83, C84: 15p, Capacitor_SMD:C_0603_1608Metric_Pad1.08x0.95mm_HandSolder, symbol Device:C
- added D10: ESD5Zxx, Diode_SMD:D_SOD-523, symbol Diode:ESD5Zxx
- added F1: 1.5A, Fuse:Fuse_1206_3216Metric, symbol Device:Polyfuse
- added L1: 3.9uH, Inductor_SMD:L_Sunlord_SWPA4030S, symbol Device:L
- added R121, R122: 5.1k, Resistor_SMD:R_0603_1608Metric_Pad0.98x0.95mm_HandSolder, symbol Device:R
- added R123: 10k, Resistor_SMD:R_0603_1608Metric_Pad0.98x0.95mm_HandSolder, symbol Device:R
- added U7: AP63203WU, Package_TO_SOT_SMD:TSOT-23-6, symbol Regulator_Switching:AP63203WU
- added U8: CH334F, Package_DFN_QFN:QFN-24-1EP_4x4mm_P0.5mm_EP2.7x2.7mm, symbol Interface_USB:CH334F
- added U9: USBLC6-2SC6, Package_TO_SOT_SMD:SOT-23-6, symbol Power_Protection:USBLC6-2SC6
- added Y3: 12MHz, Crystal:Crystal_SMD_3225-4Pin_3.2x2.5mm_HandSoldering, symbol Device:Crystal_GND24
- J1: LCSC Part (none) -> C2997433; Manufacturer_Name (none) -> HCTL; Manufacturer_Part_Number (none) -> HC-TYPE-C-16P-01A-R
Connections:
- net VBUS: now also C58.1, C61.1, C65.1, C66.1, C67.1, C68.1, C81.1, C82.1, D10.1 (K), F1.2, U7.2 (EN), U7.3 (IN), U8.19 (V5), U9.5 (VBUS); no longer J1.A4 (VBUS), J1.A9 (VBUS), J1.B4 (VBUS), J1.B9 (VBUS)
- net GND: now reaches J1.A1 (GND), J1.A12 (GND), J1.B1 (GND), J1.B12 (GND)
- net GND: now also J1.S1 (SHIELD), C58.2, C59.2, C60.2, C61.2, C63.2, C64.2, C65.2, C66.2, C67.2, C68.2, C80.2, C81.2, C82.2, C83.1, C84.1, D10.2 (A), R121.2, R122.2, U7.4 (GND), U8.25 (GND), U9.2 (GND), Y3.2 (G), Y3.4 (G)
- net CC1: now reaches J1.A5 (CC1)
- net CC1: now also R121.1
- net USB_DP: now reaches J1.A6 (D+)
- net USB_DP: now also J1.B6 (D+), U8.15 (DPU+), U9.3 (I/O2), U9.4 (I/O2)
- net USB_DM: now reaches J1.A7 (D-)
- net USB_DM: now also J1.B7 (D-), U8.14 (DMU-), U9.1 (I/O1), U9.6 (I/O1)
- net CC2: now reaches J1.B5 (CC2)
- net CC2: now also R122.1
- new net: F1.1, J1.A4 (VBUS), J1.A9 (VBUS), J1.B4 (VBUS), J1.B9 (VBUS)
- new net: C62.2, L1.1, U7.5 (SW)
- new net: C62.1, U7.6 (BST)
- new net: C84.2, U8.4 (XI), Y3.3
- new net: C83.2, U8.3 (XO), Y3.1
- new net +3.3V: C59.1, C60.1, C63.1, L1.2, U7.1 (FB)
- new net HUB_RESET: R123.2, U8.16 (~{RESET}/CDP)
- new net HUB_V33: C64.1, C80.1, R123.1, U8.20 (VDD33_{LDO})
- new net USB1_DM: U8.11 (DM1-)
- new net USB1_DP: U8.12 (DP1+)
- new net USB2_DM: U8.9 (DM2-)
- new net USB2_DP: U8.10 (DP2+)
- no-connect marks 0 -> 11
Other:
- moved on the sheet: J1

Commit message: working on the routing of the pcb
Parts:
- added R128, R129: 10k, Resistor_SMD:R_0603_1608Metric_Pad0.98x0.95mm_HandSolder, symbol Device:R
- Y3: footprint Crystal:Crystal_SMD_3225-4Pin_3.2x2.5mm_HandSoldering -> Eeloo_Pad:ABM8272T3
Connections:
- net GND: now also R129.2
- net HUB_V33: now also R128.1
- net HUB_OVCUR: now reaches U8.1 (~{OVCUR})
- net HUB_OVCUR: now also R128.2
- net HUB_PSELF: now reaches U8.18 (PSELF)
- net HUB_PSELF: now also R129.1
- no-connect marks 11 -> 9
