File: Kicad/control_module.kicad_sch (KiCad schematic)
At the start: 27 parts, among them IC3 ADS1015IDGST, IC4 PCF8575DBQR, IC5 PCF8575DBQR

Commit message: schematics correction
Parts:
- removed IC3: ADS1015IDGST, Eeloo_Pad:SOP50P490X110-10N, symbol Eeloo_Pad:ADS1015IDGST
- removed LED26, LED27, LED28, LED29, LED30, LED31, LED32, LED33, LED34, LED35, LED36: XL-5050RGBC-WS2812B, Eeloo_Pad:LED-SMD_4P-L5.0-W5.0-BL_XL-5050RGBC, symbol Eeloo_Pad:XL-5050RGBC-WS2812B
- added C34, C35, C36, C37, C38, C39, C40, C41, C42, C43, C44, C45, C85: 100n, Capacitor_SMD:C_0603_1608Metric_Pad1.08x0.95mm_HandSolder, symbol Device:C
- added C70, C71, C72, C73: 22uF, Capacitor_SMD:C_1206_3216Metric_Pad1.33x1.80mm_HandSolder, symbol Device:C
- added D7: SS34, Diode_SMD:D_SMA, symbol Diode:SS34
- added IC4: ADS7830IPWR, Eeloo_Pad:SOP65P640X120-16N, symbol Eeloo_Pad:ADS7830IPWR
- added IC6: TCA9617ADGKR, Eeloo_Pad:SOP65P490X110-8N, symbol Eeloo_Pad:PCA9617ADPJ
- added IC7: SN74AHCT1G125DBVR, Eeloo_Pad:SOT95P280X145-5N, symbol Eeloo_Pad:SN74AHCT1G125DBVR
- added J10, J11, J14, J4, J5, J6, J8, J9: Conn_01x03_Pin, Connector_JST:JST_EH_B3B-EH-A_1x03_P2.50mm_Vertical, symbol Connector:Conn_01x03_Pin
- added J3, J44, J7: Conn_01x02_Pin, Connector_JST:JST_EH_B2B-EH-A_1x02_P2.50mm_Vertical, symbol Connector:Conn_01x02_Pin
- added LED1, LED10, LED11, LED12, LED2, LED3, LED4, LED5, LED6, LED7, LED8, LED9: XL-5050RGBC-WS2812B, Eeloo_Pad:LED-SMD_4P-L5.0-W5.0-BL_XL-5050RGBC, symbol Eeloo_Pad:XL-5050RGBC-WS2812B
- added Q1: AO3400A, Package_TO_SOT_SMD:SOT-23, symbol Transistor_FET:AO3400A
- added R1, R107, R108, R109, R110, R111, R112, R113, R114, R115, R116, R117, R118, R119, R124, R125, R2, R31, R32, R33, R34, R35, R36, R37, R38, R39, R40, R41, R42, R43, R44, R45, R46, R47, R48, R49, R50, R51, R52, R53, R54, R55, R56, R57, R58, R59, R62, R65, R66, R67, R68: 10k, Resistor_SMD:R_0603_1608Metric_Pad0.98x0.95mm_HandSolder, symbol Device:R
- added R105, R106, R60, R61, R63, R64: 4k7, Resistor_SMD:R_0603_1608Metric_Pad0.98x0.95mm_HandSolder, symbol Device:R
- added R120: 100, Resistor_SMD:R_0603_1608Metric_Pad0.98x0.95mm_HandSolder, symbol Device:R
- added SW10, SW11, SW12, SW13, SW14, SW15, SW16, SW17, SW18, SW19, SW20, SW21, SW22, SW23, SW24, SW25, SW26, SW27, SW28, SW29, SW30, SW31, SW32, SW33, SW5, SW6, SW7, SW8, SW9: SW_Push, Button_Switch_SMD:SW_Push_1P1T_XKB_TS-1187A, symbol Switch:SW_Push
- IC2: renamed from IC4; value PCF8575DBQR -> PCA9535PW; footprint Eeloo_Pad:SOP64P600X175-24N -> Package_SO:TSSOP-24_4.4x7.8mm_P0.65mm; LCSC Part (none) -> C255606; Manufacturer_Name Texas Instruments -> NXP; Manufacturer_Part_Number PCF8575DBQR -> PCA9535PW,118
- IC3: renamed from IC5; value PCF8575DBQR -> PCA9535PW; footprint Eeloo_Pad:SOP64P600X175-24N -> Package_SO:TSSOP-24_4.4x7.8mm_P0.65mm; LCSC Part (none) -> C255606; Manufacturer_Name Texas Instruments -> NXP; Manufacturer_Part_Number PCF8575DBQR -> PCA9535PW,118
- LED13, LED14, LED15, LED16, LED17, LED18, LED19, LED20, LED21, LED22, LED23, LED24, LED25: Manufacturer_Name (none) -> XINGLIGHT; Manufacturer_Part_Number (none) -> XL-5050RGBC-WS2812B
Connections:
- net +5V: now also LED13.1 (VDD), LED14.1 (VDD), LED15.1 (VDD), LED16.1 (VDD), LED17.1 (VDD), LED18.1 (VDD), LED19.1 (VDD), LED20.1 (VDD), LED21.1 (VDD), LED22.1 (VDD), LED23.1 (VDD), LED24.1 (VDD), LED25.1 (VDD), C34.1, C41.1, C43.1, C44.1, C45.1, C70.1, C71.1, D7.1 (K), IC6.8 (VCC(B)), IC7.5 (VCC), J44.2 (Pin_2), LED1.1 (VDD), LED10.1 (VDD), LED11.1 (VDD), LED12.1 (VDD), LED2.1 (VDD), LED3.1 (VDD), LED4.1 (VDD), LED5.1 (VDD), LED6.1 (VDD), LED7.1 (VDD), LED8.1 (VDD), LED9.1 (VDD), R60.1, R61.1, R62.1
- net 3.3V: now also IC2.24 (VCC), IC3.24 (VCC), C35.1, C36.1, C37.1, C38.1, C39.1, C40.1, C42.1, C72.1, C73.1, C85.1, IC4.10 (REFIN/REFOUT), IC4.16 (+VDD), IC6.1 (VCC(A)), J10.1 (Pin_1), J11.1 (Pin_1), J14.1 (Pin_1), J4.1 (Pin_1), J5.1 (Pin_1), J6.1 (Pin_1), J8.1 (Pin_1), J9.1 (Pin_1), R1.2, R105.1, R106.1, R107.1, R109.1, R111.1, R113.1, R115.1, R117.1, R124.1, R125.1, R2.2, R31.1, R32.1, R33.1, R34.1, R35.1, R36.1, R37.1, R38.1, R39.1, R40.1, R41.1, R42.1, R43.1, R44.1, R45.1, R46.1, R47.1, R48.1, R49.1, R50.1, R51.1, R52.1, R53.1, R54.1, R55.1, R56.1, R57.1, R58.1, R59.1, R63.1, R64.1, R65.1, R67.1
- net at LED18.2 (DOU): now also LED23.4 (DIN)
- net GND: now reaches LED18.3 (GND)
- net GND: now also IC2.12 (GND), IC3.12 (GND), LED13.3 (GND), LED14.3 (GND), LED15.3 (GND), LED16.3 (GND), LED17.3 (GND), LED19.3 (GND), LED20.3 (GND), LED21.3 (GND), LED22.3 (GND), LED23.3 (GND), LED24.3 (GND), LED25.3 (GND), C34.2, C35.2, C36.2, C37.2, C38.2, C39.2, C40.2, C41.2, C42.2, C43.2, C44.2, C45.2, C70.2, C71.2, C72.2, C73.2, C85.2, IC4.11 (COM), IC4.9 (GND), IC6.4 (GND), IC7.1 (~{OE}), IC7.3 (GND), J10.3 (Pin_3), J11.3 (Pin_3), J14.3 (Pin_3), J3.2 (Pin_2), J4.3 (Pin_3), J5.3 (Pin_3), J6.3 (Pin_3), J7.2 (Pin_2), J8.3 (Pin_3), J9.3 (Pin_3), LED1.3 (GND), LED10.3 (GND), LED11.3 (GND), LED12.3 (GND), LED2.3 (GND), LED3.3 (GND), LED4.3 (GND), LED5.3 (GND), LED6.3 (GND), LED7.3 (GND), LED8.3 (GND), LED9.3 (GND), Q1.2 (S), R108.2, R110.2, R112.2, R114.2, R116.2, R118.2, R119.2, R66.2, R68.2, SW10.1, SW11.1, SW12.1, SW13.1, SW14.1, SW15.1, SW16.1, SW17.1, SW18.1, SW19.1, SW20.1, SW21.1, SW22.1, SW23.1, SW24.1, SW25.1, SW26.1, SW27.1, SW28.1, SW29.1, SW30.1, SW31.1, SW32.1, SW33.1, SW5.1, SW6.1, SW7.1, SW8.1, SW9.1
- net at LED18.4 (DIN): now also LED13.2 (DOU)
- net at LED24.2 (DOU): now also LED5.4 (DIN)
- net at LED24.4 (DIN): now also LED19.2 (DOU)
- net at LED25.4 (DIN): now also LED20.2 (DOU)
- net at LED22.2 (DOU): now also LED3.4 (DIN)
- net at LED22.4 (DIN): now also LED17.2 (DOU)
- net at LED21.2 (DOU): now also LED2.4 (DIN)
- net at LED21.4 (DIN): now also LED16.2 (DOU)
- net at LED16.4 (DIN): now also LED11.2 (DOU)
- net at LED20.4 (DIN): now also LED15.2 (DOU)
- net at LED19.4 (DIN): now also LED14.2 (DOU)
- net at LED15.4 (DIN): now also LED10.2 (DOU)
- net I2C_GPIO_EXT0_INT: now reaches IC2.1 (~{INT})
- net I2C_GPIO_EXT0_INT: now also R124.2
- net CTRL4: now reaches IC2.10 (P06)
- net CTRL4: now also R37.2, SW13.2
- net CTRL5: now reaches IC2.11 (P07)
- net CTRL5: now also R38.2, SW12.2
- net CTRL6: now reaches IC2.13 (P10)
- net CTRL6: now also R39.2, SW11.2
- net CTRL7: now reaches IC2.14 (P11)
- net CTRL7: now also R40.2, SW10.2
- net CTRL8: now reaches IC2.15 (P12)
- net CTRL8: now also R41.2, SW15.2
- net CTRL9: now reaches IC2.16 (P13)
- net CTRL9: now also R42.2, SW16.2
- net LIGHT: now reaches IC2.17 (P14)
- net LIGHT: now also R43.2, SW17.2
- net GEAR: now reaches IC2.18 (P15)
- net GEAR: now also R44.2, SW18.2
- net BRAKE: now reaches IC2.19 (P16)
- net BRAKE: now also R45.2, SW19.2
- net at IC2.2 (A1): now also R109.2, R110.1
- net STAGE: now reaches IC2.20 (P17)
- net STAGE: now also R59.2, SW20.2
- net at IC2.21 (A0): now also R107.2, R108.1
- net I2C0_SCL_33: now reaches IC2.22 (SCL)
- net I2C0_SCL_33: now also IC3.22 (SCL), IC4.14 (SCL), R105.2
- net I2C0_SDA_33: now reaches IC2.23 (SDA)
- net I2C0_SDA_33: now also IC3.23 (SDA), IC4.15 (SDA), R106.2
- net at IC2.3 (A2): now also R111.2, R112.1
- net SAS: now reaches IC2.4 (P00)
- net SAS: now also R31.2, SW5.2
- net RCS: now reaches IC2.5 (P01)
- net RCS: now also R32.2, SW6.2
- net CTRL0: now reaches IC2.6 (P02)
- net CTRL0: now also R33.2, SW7.2
- net CTRL1: now reaches IC2.7 (P03)
- net CTRL1: now also R34.2, SW8.2
- net CTRL2: now reaches IC2.8 (P04)
- net CTRL2: now also R35.2, SW9.2
- net CTRL3: now reaches IC2.9 (P05)
- net CTRL3: now also R36.2, SW14.2
- net I2C_GPIO_EXT1_INT: now reaches IC3.1 (~{INT})
- net I2C_GPIO_EXT1_INT: now also R125.2
- net TARGET: now reaches IC3.10 (P06)
- net TARGET: now also R52.2, SW27.2
- net ANTI_TARGET: now reaches IC3.11 (P07)
- net ANTI_TARGET: now also R53.2, SW28.2
- net MANEUVER: now reaches IC3.13 (P10)
- net MANEUVER: now also R54.2, SW33.2
- net ANTI_MANEUVER: now reaches IC3.14 (P11)
- net ANTI_MANEUVER: now also R55.2, SW32.2
- net CIBLE_ORBIT: now reaches IC3.15 (P12)
- net CIBLE_ORBIT: now also R56.2, SW31.2
- net ORBIT_SURFACE: now reaches IC3.16 (P13)
- net ORBIT_SURFACE: now also R57.2, SW30.2
- net SEA_EARTH: now reaches IC3.17 (P14)
- net SEA_EARTH: now also R58.2, SW29.2
- net JOY_BTN_D: now reaches IC3.18 (P15)
- net JOY_BTN_D: now also J7.1 (Pin_1), R2.1
- net JOY_BTN_G: now reaches IC3.19 (P16)
- net JOY_BTN_G: now also J3.1 (Pin_1), R1.1
- net at IC3.2 (A1): now also R115.2, R116.1
- net at IC3.21 (A0): now also R113.2, R114.1
- net at IC3.3 (A2): now also R117.2, R118.1
- net PROGRADE: now reaches IC3.4 (P00)
- net PROGRADE: now also R46.2, SW24.2
- net RETROGRADE: now reaches IC3.5 (P01)
- net RETROGRADE: now also R47.2, SW23.2
- net NORMAL: now reaches IC3.6 (P02)
- net NORMAL: now also R48.2, SW22.2
- net ANTINORMAL: now reaches IC3.7 (P03)
- net ANTINORMAL: now also R49.2, SW21.2
- net RADIAL_IN: now reaches IC3.8 (P04)
- net RADIAL_IN: now also R50.2, SW25.2
- net RADIAL_OUT: now reaches IC3.9 (P05)
- net RADIAL_OUT: now also R51.2, SW26.2
- net at LED17.4 (DIN): now also LED12.2 (DOU)
- net at LED14.4 (DIN): now also LED9.2 (DOU)
- net at LED13.4 (DIN): now also LED8.2 (DOU)
- net at LED23.2 (DOU): now also LED4.4 (DIN)
- new net: Q1.1 (G), R119.1, R120.2
- new net: LED3.2 (DOU), LED8.4 (DIN)
- new net: IC4.12 (A0), R67.2, R68.1
- new net: LED10.4 (DIN), LED5.2 (DOU)
- new net: LED12.4 (DIN), LED7.2 (DOU)
- new net: LED2.2 (DOU), LED7.4 (DIN)
- new net: LED11.4 (DIN), LED6.2 (DOU)
- new net: D7.2 (A), J44.1 (Pin_1), Q1.3 (D)
- new net: IC6.5 (EN), R62.2
- new net: LED4.2 (DOU), LED9.4 (DIN)
- new net: LED1.2 (DOU), LED6.4 (DIN)
- new net: IC4.13 (A1), R65.2, R66.1
- new net EXT1: IC4.1 (CH0), J14.2 (Pin_2)
- new net I2C1_SCL_33: IC6.2 (SCLA), R63.2
- new net I2C1_SCL_50: IC6.7 (SCLB), R60.2
- new net I2C1_SDA_33: IC6.3 (SDAA), R64.2
- new net I2C1_SDA_50: IC6.6 (SDAB), R61.2
- new net JOY_D_AXIS_R: IC4.3 (CH2), J10.2 (Pin_2)
- new net JOY_D_AXIS_X: IC4.5 (CH4), J8.2 (Pin_2)
- new net JOY_D_AXIS_Y: IC4.4 (CH3), J9.2 (Pin_2)
- new net JOY_G_AXIS_R: IC4.6 (CH5), J6.2 (Pin_2)
- new net JOY_G_AXIS_X: IC4.8 (CH7), J4.2 (Pin_2)
- new net JOY_G_AXIS_Y: IC4.7 (CH6), J5.2 (Pin_2)
- new net LED_CTRL_33: IC7.2 (A)
- new net LED_CTRL_50: IC7.4 (Y), LED1.4 (DIN)
- new net THROTTLE: IC4.2 (CH1), J11.2 (Pin_2)
- new net VIBRO_CTRL_33: R120.1
- no-connect marks 0 -> 22
Other:
- note added: "Button"
- note added: "EXT1"
- note added: "Joystick Droite"
- note added: "Joystick Gauche"
- note added: "Rot"
- note added: "Slider"
- note added: "Throttle"
- note added: "Vibro Connector"
- note added: "X"
- note added: "Y"
- moved on the sheet: IC2, IC3

Commit message: working on the routing of the pcb
Parts:
- added C100, C101, C102, C103, C104, C105, C106, C107, C108, C109, C110, C86, C87, C88, C89, C90, C91, C92, C93, C94, C95, C96, C97, C98, C99: 100n, Capacitor_SMD:C_0603_1608Metric_Pad1.08x0.95mm_HandSolder, symbol Device:C
- added R126: 330, Resistor_SMD:R_0603_1608Metric_Pad0.98x0.95mm_HandSolder, symbol Device:R
- added R127: 10k, Resistor_SMD:R_0603_1608Metric_Pad0.98x0.95mm_HandSolder, symbol Device:R
- LED1, LED10, LED11, LED12, LED13, LED14, LED15, LED16, LED17, LED18, LED19, LED2, LED20, LED21, LED22, LED23, LED24, LED25, LED3, LED4, LED5, LED6, LED7, LED8, LED9: footprint Eeloo_Pad:LED-SMD_4P-L5.0-W5.0-BL_XL-5050RGBC -> LED_SMD:LED_WS2812B_PLCC4_5.0x5.0mm_P3.2mm
Connections:
- net +5V: now also C100.1, C101.1, C102.1, C103.1, C104.1, C105.1, C106.1, C107.1, C108.1, C109.1, C110.1, C86.1, C87.1, C88.1, C89.1, C90.1, C91.1, C92.1, C93.1, C94.1, C95.1, C96.1, C97.1, C98.1, C99.1
- net GND: now also C100.2, C101.2, C102.2, C103.2, C104.2, C105.2, C106.2, C107.2, C108.2, C109.2, C110.2, C86.2, C87.2, C88.2, C89.2, C90.2, C91.2, C92.2, C93.2, C94.2, C95.2, C96.2, C97.2, C98.2, C99.2, R127.2
- net LED_CTRL_33: now also R127.1
- net LED_CTRL_50: now also R126.2; no longer LED1.4 (DIN)
- new net: LED1.4 (DIN), R126.1
